File: DemoNixie-KiCad/DemoNixie.kicad_pcb (KiCad board)
At the start: 4 copper layers, 275.6 x 66 mm, 122 parts, among them J1 HE10_02x10, J2 Screw_Terminal, J3 Screw_Terminal, J4 Screw_Terminal, J5 Screw_Terminal, Q1 Si9407BDY, Q2 Si9407BDY, Q3 Si9407BDY, Q4 Si9407BDY, U1 LT3746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

Commit message: finalisation controlBoard
Routing:
- net +5V: track 375.1 -> 23.9 mm, vias 17 -> 10
- net /SDI-4: track 124.7 -> 129.3 mm
- net /SCKI-4: track 128.1 -> 132.6 mm
- net /LDI-4: track 120.2 -> 124.7 mm
- net /SDI-3: track 144.2 -> 147.3 mm
- net /SCKI-3: track 147.7 -> 150.7 mm
- net /LDI-3: track 139.9 -> 142.9 mm
- net /SCKI-2: track 127.3 -> 129.8 mm
- net /SDI-2: track 124.0 -> 126.4 mm
- net /LDI-2: track 119.5 -> 121.9 mm
- net GND: vias 77 -> 87
- added copper zone on In2.Cu, net +5V
- removed copper zone on In2.Cu, net GND
Other:
- board text added: "1"
- board text added: "Arnaud Apelbaum - Antoine Bureau - Stéphane Marques - Julien Coquelet-Gaume - LPRO MECSE 2020"
- board text added: "DemoNixie"
- board text added: "LED board"
